File: electrical/v03/tpa3255-v03-overview.kicad_sch (KiCad schematic)
At the start: 180 parts, among them J1 LEFT BTL, J101 L RCA, J102 R RCA, J2 RIGHT BTL, J201 INTERNAL 48V INPUT, J202 INTERNAL 12V INPUT, J301 TRIGGER TIP / SLEEVE, J302 AUTO / COMMON / ON, J303 STATUS, J601 L XLR FEMALE, J602 R XLR FEMALE, J603 L RCA / COM / XLR, J604 R RCA / COM / XLR, J605 CHASSIS BOND, U1 TPA3255DDV, U2 NE5532, U3 NE5532, U301 VOS618A-3T, U302 SN74LVC1G14DBVR, U303 TPS3808G01DBVR, U304 SN74LVC1G17DBVR, U305 SN74LVC1G17DBVR, U306 TPS3808G01DBVR, U307 SN74LVC1G17DBVR, U4 TLV76033DBZR, U401 TPS26631PWPR, U601 INA2137UA, U602 NE5532

Commit message: Redraw the complete TPA3255 circuit with continuous signal paths
Parts:
- U1: symbol Project:TPA3255 -> Overview:TPA3255
- U601: symbol Project:INA2137 -> Overview:INA2137
Connections:
- net R_INV2: now reaches C123.1, R124.2, R125.1, U3.6 (-)
- net R_INV1: now reaches C122.1, R122.2, R123.1, U3.2 (-)
- net L_INV1: now reaches C102.1, R102.2, R103.1, U2.2 (-)
- net R_AC: now reaches C121.2, R122.1
- net L_AC: now reaches C101.2, R102.1
- net L_INV2: now reaches C103.1, R104.2, R105.1, U2.6 (-)
Other:
- note added: "12V 供電成立"
- note added: "12V 待機供電 → 類比驅動、XLR 與 3.3V 控制"
- note added: "48V 成立與延遲開聲 → RESET_N"
- note added: "48V 機內電源 → 保險絲 → 反接保護 → eFuse → 功率級 PVDD"
- note added: "AUTO / 中間 OFF / ON"
- note added: "BTL 浮接輸出：喇叭兩端均不接 GND"
- note added: "LC 輸出濾波"
- note added: "TPA3255 V0.3｜整合電路圖"
- note added: "TPA3255 偏壓、設定與本地去耦（同名標籤相連）"
- note added: "Trigger → 光耦隔離 → AUTO / OFF / ON → 電源條件判斷 → 關機保持 → 48V 開關"
- note added: "低壓音訊與控制草案；機內市電區另圖。尚未走線及實機驗證。"
- note added: "前級 Trigger 回路隔離；TRIG_RETURN 不接 GND"
- note added: "右喇叭"
- note added: "右聲道：XLR / RCA → 差動驅動"
- note added: "左喇叭"
- note added: "左聲道：XLR / RCA → 差動驅動"
- note added: "延後切斷 48V"
- note added: "所有 180 個元件皆保留。相同電源／偏壓標籤表示相連；導線交叉僅有圓點才相接。"
- note added: "濾波後回授 PFFB：由喇叭端返回 SUM_A / SUM_B"
- note added: "濾波後回授 PFFB：由喇叭端返回 SUM_C / SUM_D"
- note added: "跳線 1–2：RCA；2–3：XLR"
- note added: "音訊由左向右；四路回授繞回輸入；下方為供電與啟停控制。"
- note added: "類比中點 VMID"
- note removed: "01 平衡輸入與選擇 / XLR + RCA"
- note removed: "02 訊號驅動 / NE5532"
- note removed: "03 濾波後回授 / PFFB"
- note removed: "04 功率放大與喇叭輸出 / TPA3255 + LC"
- note removed: "05 類比供電與去耦 / 12V + VMID"
- note removed: "06 控制供電與狀態 / 3.3V"
- note removed: "07 自動啟停與關機延遲 / Trigger"
- note removed: "08 主電源開關與靜音 / 48V + RESET"
- note removed: "AUX_GOOD falls first to mute. HOLD_CAP keeps main DC on briefly; verify timing on hardware."
- note removed: "Buffered REF; C607 at U601, C608 at U602. Pin 1 / shells bond to chassis at entry."
- note removed: "C209 / C210 at GVDD_AB / GVDD_CD separately."
- note removed: "C310-C315: one at each U302-U307 VCC/VDD pin on PCB."
- note removed: "C601/C602 and C603/C604: match pairs to 1% measured capacitance."
- note removed: "DVDD / AVDD / VBG: internal outputs, bypass only."
- note removed: "Design input: 9-15V DC, nominal 12V. Verify Z10 voltage, polarity and drive capability before connecting."
- note removed: "External SPDT centre-OFF switch."
- note removed: "Fit all four feedback branches; do not substitute R/C values without a loop review."
- note removed: "High-impedance monitoring only; no external 5V pullups."
- note removed: "INPUT SUPPLY / VMID"
- note removed: "Internal AC/DC modules share one mains inlet. Trigger-off disconnects PVDD; 12V standby remains on."
- note removed: "Internal balanced-to-single-ended receiver; this is not a fully differential end-to-end amplifier."
- note removed: "J603/J604: fit 2-3 for XLR, 1-2 for RCA. Change both only in standby."
- note removed: "M1=M2=0; OSC pins intentionally NC."
- note removed: "MODE open: latch fault; cycle Trigger to retry."
- note removed: "Matching net labels connect throughout this single page."
- note removed: "NE5532 on 12V, VMID approx. 6V. Signal capacitors are bipolar/film."
- note removed: "No external reverse-block FET. Surge testing pending."
- note removed: "PFFB + LC: hardware loop stability still needs testing."
- note removed: "PFFB summing resistors BEFORE AC coupling; Z10 RCA 2.5Vrms target"
- note removed: "PFFB, input bandwidth and LC are one loop: reduced model is NOT hardware stability proof."
- note removed: "PVDD >40.9V, then ~1.03s delay."
- note removed: "PVDD from section 08. 12V standby remains on; no mains wiring on this PCB."
- note removed: "Place 2x MLCC + 1x bulk at EACH PVDD group."
- note removed: "Same-arm negative feedback: SPK_A to SUM_A, etc. Summing node is BEFORE the input coupling capacitor."
- note removed: "Speaker terminals float: never join B or D to GND."
- note removed: "TPA fault protection remains internal; no automatic fault retry loop."
- note removed: "TPA3255 V0.3 完整電路總圖"
- note removed: "TRIG_RETURN is isolated from GND and chassis. Use an insulated jack; no trigger-powered relay coil."
- note removed: "Top PowerPAD: ground heatsink per TI pin table."
- note removed: "Trigger OFF enters standby, not AC mains isolation."
- note removed: "XLR female: 1 shield, 2 hot, 3 cold. Both signal legs are AC coupled; do not ground pin 3."
- note removed: "低壓音訊與控制草案；機內市電區另圖規劃。尚未完成走線及實機驗證。"
- note removed: "供電／控制：05 類比供電、06 控制供電；07 Trigger → 08 電源開關／RESET → 04 功率級。"
- note removed: "同名網路標籤表示相連。180 個元件完整保留；A0 單頁，可放大閱讀。"
- note removed: "音訊：01 輸入 → 02 驅動 → 04 功率輸出；03 回授由輸出返回輸入。"
- title: TPA3255 V0.3 / COMPLETE SINGLE-PAGE SCHEMATIC -> TPA3255 V0.3 / INTEGRATED CIRCUIT
- moved on the sheet: C1, C10, C101, C102, C103, C11, C12, C121, C122, C123, C13, C14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
